File: Pcb/hiro.kicad_pcb (KiCad board)
At the start: 2 copper layers, 80.1 x 107.1 mm, 17 parts, among them J1 Micro_SD_Card_Det_Hirose_DM3AT, J2 AudioJack3, J3 Conn_01x08, J4 Conn_01x02, SW1 RotaryEncoder_Switch, U1 XIAO-ESP32-S3-Plus-SMD, U2 PCM5102A, U3 MAX98357A

Commit message: Final PCB (rev1)
Parts:
- moved SW1 0.50 mm to (169.0, 91.7)
Routing:
- net /SW1: track 45.9 -> 82.8 mm, vias 0 -> 2
- net +3.3V: track 101.1 -> 78.1 mm
- net (no net): track 0.00 -> 8.49 mm
Other:
- board text added: "H.I.R.O. Rev1"
Changed lines of the file:
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@@
 	(footprint "Libs:Right angle EC11 Rotary Encoder"
 		(layer "F.Cu")
-		(at 168.504935 91.736455 90)
+		(at 169.004935 91.736455 90)
 		(property "Reference" "SW1"
 			(at 0 -0.5 90)
@@
 		(layer "Edge.Cuts")
 	)
+	(gr_text "H.I.R.O. Rev1\n"
+		(at 187.25 190 0)
+		(layer "Edge.Cuts")
+		(effects
+			(font
+				(size 1 1)
+				(thickness 0.15)
+			)
+			(justify left bottom)
+		)
+	)
+	(segment
+		(start 152 81)
+		(end 158 87)
+		(width 0.2)
+		(layer "F.Cu")
+		(net "")
+	)
 	(segment
 		(start 144.252548 134.8)
@@
 	)
 	(segment
+		(start 144.17 56.17)
+		(end 145 57)
+		(width 0.2)
+		(layer "F.Cu")
+		(net "+3.3V")
+	)
+	(segment
 		(start 117.8125 137.225)
 		(end 117.156544 137.225)
@@
 	)
 	(segment
+		(start 96.99 56.17)
+		(end 144.17 56.17)
+		(width 0.2)
+		(layer "F.Cu")
+		(net "+3.3V")
+	)
+	(segment
 		(start 146.9375 133.1125)
 		(end 146.9375 132.6125)
@@
 	)
 	(segment
-		(start 121.82 80.18)
-		(end 121 80.18)
-		(width 0.2)
-		(layer "F.Cu")
-		(net "+3.3V")
-	)
-	(segment
 		(start 122.775 134.0875)
 		(end 122 134.8625)
@@
 	)
 	(segment
-		(start 96.99 56.17)
-		(end 121 80.18)
-		(width 0.2)
-		(layer "F.Cu")
-		(net "+3.3V")
-	)
-	(segment
 		(start 116.775 132.345778)
 		(end 117.745778 131.375)
@@
 		(net "+3.3V")
 	)
-	(segment
-		(start 121 80.18)
-		(end 121 84)
-		(width 0.2)
-		(layer "F.Cu")
-		(net "+3.3V")
-	)
-	(segment
-		(start 145 57)
-		(end 121.82 80.18)
-		(width 0.2)
-		(layer "F.Cu")
-		(net "+3.3V")
-	)
 	(via
 		(at 145 57)
@@
 	)
 	(segment
+		(start 160 80)
+		(end 166.98925 73.01075)
+		(width 0.2)
+		(layer "F.Cu")
+		(net "/SW1")
+	)
+	(segment
+		(start 153.565685 87)
+		(end 154 87)
+		(width 0.2)
+		(layer "F.Cu")
+		(net "/SW1")
+	)
+	(segment
 		(start 132.236012 132.572567)
 		(end 139.295012 125.513567)
@@
 	)
 	(segment
+		(start 166.98925 73.01075)
+		(end 167.554935 73.01075)
+		(width 0.2)
+		(layer "F.Cu")
+		(net "/SW1")
+	)
+	(segment
 		(start 139.295012 98.696378)
 		(end 141.869307 98.696378)
@@
 	)
 	(segment
+		(start 141.869307 98.696378)
+		(end 153.565685 87)
+		(width 0.2)
+		(layer "F.Cu")
+		(net "/SW1")
+	)
+	(segment
 		(start 131.086012 136.073823)
 		(end 132.236012 134.923823)
@@
 		(net "/SW1")
 	)
+	(via
+		(at 154 87)
+		(size 0.6)
+		(drill 0.3)
+		(layers "F.Cu" "B.Cu")
+		(net "/SW1")
+	)
+	(via
+		(at 160 80)
+		(size 0.6)
+		(drill 0.3)
+		(layers "F.Cu" "B.Cu")
+		(net "/SW1")
+	)
+	(segment
+		(start 154 86)
+		(end 160 80)
+		(width 0.2)
+		(layer "B.Cu")
+		(net "/SW1")
+	)
+	(segment
+		(start 154 87)
+		(end 154 86)
+		(width 0.2)
+		(layer "B.Cu")
+		(net "/SW1")
+	)

Commit message: moved speaker
It now lines up with the like left square thingy in the art.
Parts:
- moved LS1 12.6 mm to (104.0, 100.0)
Routing:
- net Net-(U3-OUTP): track 55.6 -> 68.8 mm
- net Net-(U3-OUTN): track 48.8 -> 61.9 mm
Changed lines of the file:
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@@
 	(footprint "Spkr:SPKR_CVS-1708"
 		(layer "F.Cu")
-		(at 102.6 112.55)
+		(at 104 100)
 		(property "Reference" "LS1"
 			(at -0.637345 -9.560295 0)
@@
 	)
 	(segment
-		(start 98.8 112.55)
+		(start 98.875 112.625)
 		(end 118.175 131.925)
 		(width 0.2)
@@
 	)
 	(segment
+		(start 98.8 112.55)
+		(end 98.875 112.625)
+		(width 0.2)
+		(layer "B.Cu")
+		(net "Net-(U3-OUTP)")
+	)
+	(segment
+		(start 98.875 112.625)
+		(end 100.2 111.3)
+		(width 0.2)
+		(layer "B.Cu")
+		(net "Net-(U3-OUTP)")
+	)
+	(segment
+		(start 100.2 111.3)
+		(end 100.2 100)
+		(width 0.2)
+		(layer "B.Cu")
+		(net "Net-(U3-OUTP)")
+	)
+	(segment
 		(start 118.175 131.925)
 		(end 146.375 131.925)
@@
 	)
 	(segment
+		(start 106.425 101.375)
+		(end 107.8 100)
+		(width 0.2)
+		(layer "B.Cu")
+		(net "Net-(U3-OUTN)")
+	)
+	(segment
 		(start 145 131)
 		(end 123.151471 131)
@@
 	)
 	(segment
+		(start 106.425 112.575)
+		(end 106.425 101.375)
+		(width 0.2)
+		(layer "B.Cu")
+		(net "Net-(U3-OUTN)")
+	)
+	(segment
 		(start 120.4 126.55)
+		(end 106.425 112.575)
+		(width 0.2)
+		(layer "B.Cu")
+		(net "Net-(U3-OUTN)")
+	)
+	(segment
+		(start 106.425 112.575)
 		(end 106.4 112.55)
 		(width 0.2)

Commit message: Some changes i forget
Parts:
- moved LS1 2.50 mm to (101.5, 100.0)
Routing:
- net (no net): track 8.49 -> 0.00 mm
- net GND: vias 10 -> 8
Other:
- board text removed: "H.I.R.O. Rev1"
Changed lines of the file:
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@@
 	(footprint "Spkr:SPKR_CVS-1708"
 		(layer "F.Cu")
-		(at 104 100)
+		(at 101.5 100)
 		(property "Reference" "LS1"
 			(at -0.637345 -9.560295 0)
@@
 		(layer "Edge.Cuts")
 	)
-	(gr_text "H.I.R.O. Rev1\n"
-		(at 187.25 190 0)
-		(layer "Edge.Cuts")
-		(effects
-			(font
-				(size 1 1)
-				(thickness 0.15)
-			)
-			(justify left bottom)
-		)
-	)
-	(segment
-		(start 152 81)
-		(end 158 87)
-		(width 0.2)
-		(layer "F.Cu")
-		(net "")
-	)
 	(segment
 		(start 144.252548 134.8)
@@
 	)
 	(via
-		(at 108.5 139.825)
-		(size 0.6)
-		(drill 0.3)
-		(layers "F.Cu" "B.Cu")
-		(net "GND")
-	)
-	(via
 		(at 112.0875 135.225)
 		(size 0.6)
@@
 	)
 	(via
-		(at 108.5 137.825)
-		(size 0.6)
-		(drill 0.3)
-		(layers "F.Cu" "B.Cu")
-		(net "GND")
-	)
-	(via
 		(at 144.881276 136.881276)
 		(size 0.6)
@@
 	)
 	(segment
-		(start 98.875 112.625)
-		(end 118.175 131.925)
-		(width 0.2)
-		(layer "B.Cu")
-		(net "Net-(U3-OUTP)")
-	)
-	(segment
-		(start 98.8 112.55)
-		(end 98.875 112.625)
-		(width 0.2)
-		(layer "B.Cu")
-		(net "Net-(U3-OUTP)")
-	)
-	(segment
-		(start 98.875 112.625)
-		(end 100.2 111.3)
+		(start 118.175 131.925)
+		(end 146.375 131.925)
 		(width 0.2)
 		(layer "B.Cu")
@@
 	)
 	(segment
-		(start 100.2 111.3)
-		(end 100.2 100)
+		(start 97.7 100)
+		(end 97.7 111.45)
 		(width 0.2)
 		(layer "B.Cu")
@@
 	)
 	(segment
-		(start 118.175 131.925)
-		(end 146.375 131.925)
+		(start 97.7 111.45)
+		(end 118.175 131.925)
 		(width 0.2)
 		(layer "B.Cu")
@@
 	)
 	(segment
-		(start 106.425 101.375)
-		(end 107.8 100)
+		(start 145 131)
+		(end 123.151471 131)
 		(width 0.2)
 		(layer "B.Cu")
@@
 	)
 	(segment
-		(start 145 131)
-		(end 123.151471 131)
+		(start 120.4 126.55)
+		(end 106.425 112.575)
 		(width 0.2)
 		(layer "B.Cu")
@@
 	(segment
 		(start 106.425 112.575)
-		(end 106.425 101.375)
+		(end 106.4 112.55)
 		(width 0.2)
 		(layer "B.Cu")
@@
 	)
 	(segment
-		(start 120.4 126.55)
-		(end 106.425 112.575)
+		(start 123.151471 131)
+		(end 120.4 128.248529)
 		(width 0.2)
 		(layer "B.Cu")
@@
 	(segment
 		(start 106.425 112.575)
-		(end 106.4 112.55)
+		(end 106.425 101.125)
 		(width 0.2)
 		(layer "B.Cu")
@@
 	)
 	(segment
-		(start 123.151471 131)
-		(end 120.4 128.248529)
+		(start 106.425 101.125)
+		(end 105.3 100)
 		(width 0.2)
 		(layer "B.Cu")

Commit message: FINAL PCB FINAL PCB FINAL PCB
Parts:
- added R1: 1M, Resistor_SMD:R_0603_1608Metric_Pad0.98x0.95mm_HandSolder, F.Cu at (146.5, 137.2)
Connections:
- J3 pad 3: /DIN1 -> /MOSI
- J3 pad 7: /MOSI -> /LCD_RST
- J3 pad 8: /MISO -> /LCD_BL
- U1 pad 25: /SW3 -> unconnected-(U1-GPIO40_MTDO_CAM_SDA_I2S_WS-Pad25)
- U1 pad 29: /SW1 -> unconnected-(U1-GPIO39_MTCK_CAM_SCL_I2S_SCK-Pad29)
- U1 pad 3: unconnected-(U1-GPIO3_A2_D2-Pad3) -> /SW1
- U1 pad 4: unconnected-(U1-GPIO4_A3_D3-Pad4) -> /SW3
- U1 pad 5: unconnected-(U1-GPIO5_A4_D4_SDA-Pad5) -> /LCD_RST
- U1 pad 6: unconnected-(U1-GPIO6_A5_D5_SCL-Pad6) -> /LCD_BL
- U2 pad 12: unconnected-(U2-SCK-Pad12) -> GND
- U3 pad 4: unconnected-(U3-~{SD_MODE}-Pad4) -> /SD_MODE
Routing:
- net /DIN1: track 107.5 -> 21.6 mm, vias 3 -> 2
- net /LCD_RST: track 0.00 -> 78.7 mm, vias 0 -> 1
- net /LCD_BL: track 0.00 -> 73.2 mm, vias 0 -> 1
- net +3.3V: track 78.1 -> 125.4 mm, vias 2 -> 7
- net GND: track 168.4 -> 134.4 mm, vias 8 -> 6
- net /SCK: track 128.8 -> 162.4 mm, vias 2 -> 1
- net /MISO: track 129.2 -> 101.5 mm, vias 2 -> 0
- net /SW3: track 73.8 -> 52.8 mm
- net /MOSI: track 136.4 -> 122.9 mm, vias 2 -> 1
- net Net-(U3-OUTN): track 61.8 -> 55.4 mm
- net /CS1: track 98.2 -> 91.8 mm, vias 0 -> 2
- net Net-(U3-OUTP): track 68.6 -> 62.9 mm
- net /ENCB: track 62.8 -> 67.3 mm, vias 2 -> 1
- net /DC: track 76.7 -> 73.0 mm
- net /SW2: track 50.3 -> 47.0 mm, vias 0 -> 2
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