File: Pcb/hiro.kicad_sch (KiCad schematic)
At the start: 17 parts, among them J1 Micro_SD_Card_Det_Hirose_DM3AT, J2 AudioJack3, J3 Conn_01x08, J4 Conn_01x02, SW1 RotaryEncoder_Switch, U1 XIAO-ESP32-S3-Plus-SMD, U2 PCM5102A, U3 MAX98357A

Commit message: FINAL PCB FINAL PCB FINAL PCB
Parts:
- added R1: 1M, Resistor_SMD:R_0603_1608Metric_Pad0.98x0.95mm_HandSolder, symbol Device:R
Connections:
- net +3.3V: now also R1.1
- net DIN1: no longer J3.3 (Pin_3)
- net GND: now also U2.12 (SCK)
- net MISO: no longer J3.8 (Pin_8)
- net MOSI: now also J3.3 (Pin_3); no longer J3.7 (Pin_7)
- net SW1: now also U1.3 (GPIO3_A2_D2); no longer U1.29 (GPIO39_MTCK_CAM_SCL_I2S_SCK)
- net SW3: now also U1.4 (GPIO4_A3_D3); no longer U1.25 (GPIO40_MTDO_CAM_SDA_I2S_WS)
- net SD_MODE: now reaches U3.4 (~{SD_MODE})
- net SD_MODE: now also R1.2
- net LCD_RST: now reaches U1.5 (GPIO5_A4_D4_SDA)
- net LCD_RST: now also J3.7 (Pin_7)
- net LCD_BL: now reaches U1.6 (GPIO6_A5_D5_SCL)
- net LCD_BL: now also J3.8 (Pin_8)
- no-connect marks 21 -> 17
